File: pcb/TP_Final.sch (KiCad schematic (older format))
At the start: 20 parts, among them J1 A, J2 B, Q1 DMN2058U, U1 MQ-137, U2 MCP3551, U3 TXB0106

Commit message: Inicio PCB - Posicionamiento de componentes
Parts:
- C1: footprint Fiducial:Fiducial_0.75mm_Mask1.5mm -> Capacitor_SMD:C_0805_2012Metric
Changed lines of the file:
@@
 F 0 "C1" H 4800 2850 50  0000 C CNN
 F 1 "100n" H 4850 2750 50  0000 C CNN
-F 2 "Fiducial:Fiducial_0.75mm_Mask1.5mm" H 4550 2800 50  0001 C CNN
+F 2 "Capacitor_SMD:C_0805_2012Metric" H 4550 2800 50  0001 C CNN
 F 3 "https://ar.mouser.com/datasheet/2/212/KEM_C1002_X7R_SMD-1102033.pdf" H 4550 2800 50  0001 C CNN
 F 4 "80-C0805C104M5R" H 4550 2800 50  0001 C CNN "Código Mouser"

Commit message: Actualizo PCB
Connections:
- net +5V: now also U1.4 (A2), U1.5 (VH-); no longer U1.2 (VH+), U1.6 (A1)
- net at JP2.2 (Pin_2), R2.1: now also U1.3 (B2); no longer U1.1 (B1)
- net at Q1.3 (D): now also U1.2 (VH+); no longer U1.5 (VH-)
- removed net NC: J1.2 (Pin_2), J1.6 (Pin_6), J2.2 (Pin_2), J2.3 (Pin_3), J2.4 (Pin_4), J2.5 (Pin_5), J2.6 (Pin_6)
- no-connect marks 8 -> 15
Changed lines of the file:
@@
 	0    -1   -1   0
-$EndComp
-$Comp
-L tp_final_symbols:MQ-137 U1
-U 1 1 61370CE5
-P 1700 3600
-F 0 "U1" H 1850 4050 50  0000 C CNN
-F 1 "MQ-137" H 1950 3950 50  0000 C CNN
-F 2 "Sensor:MQ-6" H 1750 3150 50  0001 C CNN
-F 3 "https://www.winsen-sensor.com/d/files/semiconductor/mq137.pdf" H 1700 3850 50  0001 C CNN
-F 4 "474-SEN-17053" H 1700 3600 50  0001 C CNN "Código Mouser"
-	1    1700 3600
-	1    0    0    -1
 $EndComp
 Wire Wire Line
@@
 Text Label 10000 3400 2    50   ~ 0
 PWM
-Text Label 9950 3600 2    50   ~ 0
-NC
 Text Label 8950 4100 0    50   ~ 0
 GND
 Text Label 8900 4000 0    50   ~ 0
 +3.3V
-Text Label 8950 3900 0    50   ~ 0
-NC
 Text Label 8950 3800 0    50   ~ 0
 MISO
@@
 Text Label 8950 3600 0    50   ~ 0
 CS
-Text Label 8950 3500 0    50   ~ 0
-NC
 Text Label 8950 3400 0    50   ~ 0
 AN
-Text Label 9950 3700 2    50   ~ 0
-NC
-Text Label 9950 3800 2    50   ~ 0
-NC
 Text Label 10000 4000 2    50   ~ 0
 +5V
@@
 Text Notes 7450 4900 0    50   ~ 0
 Ajusta niveles\nde tensión
-Text Label 9950 3900 2    50   ~ 0
-NC
 $Comp
 L power:+5V #PWR0113
@@
 Wire Wire Line
 	9800 4100 10250 4100
-Text Label 9950 3500 2    50   ~ 0
-NC
 Wire Wire Line
 	9800 3500 9950 3500
@@
 	1    0    0    -1
 $EndComp
+$Comp
+L tp_final_symbols:MQ-137 U1
+U 1 1 61370CE5
+P 1700 3600
+F 0 "U1" H 1850 4050 50  0000 C CNN
+F 1 "MQ-137" H 1950 3950 50  0000 C CNN
+F 2 "Sensor:MQ-6" H 1750 3150 50  0001 C CNN
+F 3 "https://www.winsen-sensor.com/d/files/semiconductor/mq137.pdf" H 1700 3850 50  0001 C CNN
+F 4 "474-SEN-17053" H 1700 3600 50  0001 C CNN "Código Mouser"
+	1    1700 3600
+	1    0    0    1
+$EndComp
+NoConn ~ 9950 3500
+NoConn ~ 9950 3600
+NoConn ~ 9950 3700
+NoConn ~ 9950 3800
+NoConn ~ 9950 3900
+NoConn ~ 8950 3900
+NoConn ~ 8950 3500
 $EndSCHEMATC
